File: pollen_controller_pcb/pollen_controller_pcb.kicad_pcb (KiCad board)
At the start: 2 copper layers, 15 parts, among them J1 Conn_02x20_Odd_Even, J2 Motor focus, J3 Motor tape, J4 Focus sensor, J5 Lights, J6 Power in, J7 GPS, U1 ULN2003, U2 ULN2003, U3 NB-IOT-BC660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

Commit message: PCB changes
Parts:
- added J8: Status LED, Connector_PinSocket_2.54mm:PinSocket_1x02_P2.54mm_Vertical, F.Cu at (44.8, 24.5)
- added R5: 100, Resistor_THT:R_Axial_DIN0207_L6.3mm_D2.5mm_P10.16mm_Horizontal, F.Cu at (45.6, 20.0)
- J2, J3: footprint Connector_PinHeader_2.54mm:PinHeader_1x04_P2.54mm_Vertical -> Connector_PinHeader_2.54mm:PinHeader_1x05_P2.54mm_Vertical
- moved R3 44.3 mm to (41.2, 34.9), turned to -90 degrees
- moved R4 41.1 mm to (45.0, 45.1), turned to 90 degrees
- moved R2 36.1 mm to (32.8, 27.7), turned to -90 degrees
- moved R1 35.2 mm to (32.5, 25.1), turned to 90 degrees
- moved U2 33.1 mm to (62.2, 79.3)
- moved J7 32.7 mm to (49.0, 24.4)
- moved U4 31.2 mm to (119.7, 21.4)
- moved J6 30.8 mm to (36.3, 24.5)
- moved U1 28.9 mm to (37.2, 79.5)
- moved J2 26.4 mm to (74.2, 79.5)
- moved U3 26.4 mm to (62.6, 54.9)
- moved J3 24.0 mm to (49.4, 79.5)
- moved J5 22.6 mm to (40.5, 24.5)
- moved J4 7.70 mm to (53.2, 24.5)
Connections:
- J1 pad 10: unconnected-(J1-Pin_10-Pad10) -> /NB-IOT_TX
- J1 pad 11: unconnected-(J1-Pin_11-Pad11) -> /FOCUS_SENSOR
- J1 pad 13: unconnected-(J1-Pin_13-Pad13) -> /NB-IOT_RST
- J1 pad 17: unconnected-(J1-Pin_17-Pad17) -> +3.3V
- J1 pad 22: unconnected-(J1-Pin_22-Pad22) -> /DHT
- J1 pad 29: unconnected-(J1-Pin_29-Pad29) -> /GPS_TX
- J1 pad 31: unconnected-(J1-Pin_31-Pad31) -> /MOTOR_FOCUS_1
- J1 pad 32: unconnected-(J1-Pin_32-Pad32) -> /MOTOR_TAPE_4
- J1 pad 33: unconnected-(J1-Pin_33-Pad33) -> /MOTOR_FOCUS_2
- J1 pad 35: unconnected-(J1-Pin_35-Pad35) -> /MOTOR_FOCUS_3
- J1 pad 36: unconnected-(J1-Pin_36-Pad36) -> /MOTOR_TAPE_3
- J1 pad 37: unconnected-(J1-Pin_37-Pad37) -> /MOTOR_FOCUS_4
- J1 pad 38: unconnected-(J1-Pin_38-Pad38) -> /MOTOR_TAPE_2
- J1 pad 40: unconnected-(J1-Pin_40-Pad40) -> /MOTOR_TAPE_1
- J1 pad 7: unconnected-(J1-Pin_7-Pad7) -> /STATUS_LED
- J1 pad 8: unconnected-(J1-Pin_8-Pad8) -> /NB-IOT_RX
- J2 pad 1: unconnected-(J2-Pin_1-Pad1) -> Net-(J2-Pin_1)
- J2 pad 2: unconnected-(J2-Pin_2-Pad2) -> Net-(J2-Pin_2)
- J2 pad 3: unconnected-(J2-Pin_3-Pad3) -> Net-(J2-Pin_3)
- J2 pad 4: unconnected-(J2-Pin_4-Pad4) -> Net-(J2-Pin_4)
- J3 pad 1: unconnected-(J3-Pin_1-Pad1) -> Net-(J3-Pin_1)
- J3 pad 2: unconnected-(J3-Pin_2-Pad2) -> Net-(J3-Pin_2)
- J3 pad 3: unconnected-(J3-Pin_3-Pad3) -> Net-(J3-Pin_3)
- J3 pad 4: unconnected-(J3-Pin_4-Pad4) -> Net-(J3-Pin_4)
- U1 pad 1: unconnected-(U1-I1-Pad1) -> /MOTOR_TAPE_1
- U1 pad 13: unconnected-(U1-O4-Pad13) -> Net-(J3-Pin_4)
- U1 pad 14: unconnected-(U1-O3-Pad14) -> Net-(J3-Pin_3)
- U1 pad 15: unconnected-(U1-O2-Pad15) -> Net-(J3-Pin_2)
- U1 pad 16: unconnected-(U1-O1-Pad16) -> Net-(J3-Pin_1)
- U1 pad 2: unconnected-(U1-I2-Pad2) -> /MOTOR_TAPE_2
- U1 pad 3: unconnected-(U1-I3-Pad3) -> /MOTOR_TAPE_3
- U1 pad 4: unconnected-(U1-I4-Pad4) -> /MOTOR_TAPE_4
- U1 pad 8: unconnected-(U1-GND-Pad8) -> GND
- U1 pad 9: unconnected-(U1-COM-Pad9) -> +5V
- U2 pad 1: unconnected-(U2-I1-Pad1) -> /MOTOR_FOCUS_1
- U2 pad 13: unconnected-(U2-O4-Pad13) -> Net-(J2-Pin_4)
- U2 pad 14: unconnected-(U2-O3-Pad14) -> Net-(J2-Pin_3)
- U2 pad 15: unconnected-(U2-O2-Pad15) -> Net-(J2-Pin_2)
- U2 pad 16: unconnected-(U2-O1-Pad16) -> Net-(J2-Pin_1)
- U2 pad 2: unconnected-(U2-I2-Pad2) -> /MOTOR_FOCUS_2
- U2 pad 3: unconnected-(U2-I3-Pad3) -> /MOTOR_FOCUS_3
- U2 pad 4: unconnected-(U2-I4-Pad4) -> /MOTOR_FOCUS_4
- U2 pad 8: unconnected-(U2-GND-Pad8) -> GND
- U2 pad 9: unconnected-(U2-COM-Pad9) -> +5V
- U3 pad 19: unconnected-(U3-RxD-Pad19) -> /NB-IOT_RX
- U3 pad 20: unconnected-(U3-TxD-Pad20) -> /NB-IOT_TX
- U3 pad 3: unconnected-(U3-VCC-Pad3) -> +3.3V
- U3 pad 4: unconnected-(U3-GND-Pad4) -> GND
- U3 pad 9: unconnected-(U3-RST-Pad9) -> /NB-IOT_RST
- U4 pad 1: unconnected-(U4-VDD-Pad1) -> +3.3V
- U4 pad 2: unconnected-(U4-SDA-Pad2) -> /DHT
- U4 pad 3: Net-(U4-GND-Pad3) -> GND
- U4 pad 4: Net-(U4-GND-Pad3) -> GND
Routing:
- net /NB-IOT_TX: track 0.00 -> 119.4 mm
- net /NB-IOT_RX: track 0.00 -> 101.5 mm
- net /FOCUS_SENSOR: track 0.00 -> 68.2 mm
- net /NB-IOT_RST: track 0.00 -> 46.8 mm
- net +5V: track 0.00 -> 40.3 mm
- net +3.3V: track 0.00 -> 33.0 mm
- net Net-(J4-Pin_2): track 0.00 -> 29.4 mm
- net /STATUS_LED: track 0.00 -> 17.6 mm
- net GND: track 0.00 -> 5.30 mm
- net Net-(J8-Pin_1): track 0.00 -> 4.83 mm

Commit message: PCB changes
Parts:
- added J9: Fan, Connector_PinSocket_2.54mm:PinSocket_1x03_P2.54mm_Vertical, F.Cu at (33.2, 61.2)
- added Q1: PN2222A, Package_TO_SOT_THT:TO-92L_HandSolder, F.Cu at (32.7, 56.9)
- added R6: 4k7, Resistor_THT:R_Axial_DIN0207_L6.3mm_D2.5mm_P10.16mm_Horizontal, F.Cu at (32.8, 42.7)
- moved U4 121.6 mm to (17.4, 87.1)
Connections:
- J1 pad 15: unconnected-(J1-Pin_15-Pad15) -> /FAN_CONTROL
Routing:
- net Net-(J9-Pin_3): track 0.00 -> 5.64 mm
- net /FAN_CONTROL: track 0.00 -> 3.70 mm
- net Net-(Q1-B): track 0.00 -> 3.28 mm
- net GND: track 5.30 -> 6.84 mm
